File: hardware/net-bmp/ethernet.kicad_sch (KiCad schematic)
At the start: 24 parts, among them J7 HR911105A, U4 LAN8742A

Commit message: chore: build with stubs
Parts:
- added R9: 10k, Resistor_SMD:R_0402_1005Metric, symbol Device:R
Connections:
- net GND: now also R9.1
- net LED2: now also R9.2
Changed lines of the file:
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@@
   (title_block
     (title "net-bmp")
-    (date "2023-10-31")
-    (rev "a")
+    (date "2023-11-11")
+    (rev "b")
     (company "elagil")
   )
@@
   )
   (junction (at 109.22 46.99) (diameter 0) (color 0 0 0 0)
+  )
+  (junction (at 147.32 114.3) (diameter 0) (color 0 0 0 0)
   )
   (junction (at 185.42 34.29) (diameter 0) (color 0 0 0 0)
@@
     (stroke (width 0) (type default))
   )
+  (wire (pts (xy 147.32 114.3) (xy 149.86 114.3))
+    (stroke (width 0) (type default))
+  )
   (wire (pts (xy 165.1 49.53) (xy 165.1 55.88))
     (stroke (width 0) (type default))
@@
     (stroke (width 0) (type default))
   )
-  (wire (pts (xy 142.24 114.3) (xy 149.86 114.3))
+  (wire (pts (xy 142.24 114.3) (xy 147.32 114.3))
     (stroke (width 0) (type default))
   )
@@
     (stroke (width 0) (type default))
   )
+  (wire (pts (xy 147.32 124.46) (xy 147.32 134.62))
+    (stroke (width 0) (type default))
+  )
   (wire (pts (xy 83.82 72.39) (xy 80.01 72.39))
     (stroke (width 0) (type default))
@@
   )
   (wire (pts (xy 102.87 43.18) (xy 102.87 46.99))
+    (stroke (width 0) (type default))
+  )
+  (wire (pts (xy 147.32 114.3) (xy 147.32 116.84))
     (stroke (width 0) (type default))
   )
@@
     )
   )
+  (symbol (lib_id "power:GND") (at 147.32 134.62 0) (unit 1)
+    (in_bom yes) (on_board yes) (dnp no) (fields_autoplaced)
+    (property "Reference" "#PWR047" (at 147.32 140.97 0)
+      (effects (font (size 1.27 1.27)) hide)
+    )
+    (property "Value" "GND" (at 147.32 139.7 0)
+      (effects (font (size 1.27 1.27)))
+    )
+    (property "Footprint" "" (at 147.32 134.62 0)
+      (effects (font (size 1.27 1.27)) hide)
+    )
+    (property "Datasheet" "" (at 147.32 134.62 0)
+      (effects (font (size 1.27 1.27)) hide)
+    )
+    (pin "1")
+    (instances
+      (project "net-bmp"
+        (path "/0556e588-02fe-48e5-93e8-fa3aab1c90e7"
+          (reference "#PWR047") (unit 1)
+        )
+        (path "/0556e588-02fe-48e5-93e8-fa3aab1c90e7/05fc74b7-f058-42ca-bffa-27bc74c664f2"
+          (reference "#PWR087") (unit 1)
+        )
+      )
+    )
+  )
   (symbol (lib_id "Device:C") (at 139.7 39.37 0) (unit 1)
     (in_bom yes) (on_board yes) (dnp no)
@@
         )
       )
+    )
+  )
+  (symbol (lib_id "Device:R") (at 147.32 120.65 0) (mirror x) (unit 1)
+    (in_bom yes) (on_board yes) (dnp no)
+    (property "Reference" "R9" (at 144.78 119.38 0)
+      (effects (font (size 1.27 1.27)) (justify right))
+    )
+    (property "Value" "10k" (at 144.78 121.92 0)
+      (effects (font (size 1.27 1.27)) (justify right))
+    )
+    (property "Footprint" "Resistor_SMD:R_0402_1005Metric" (at 145.542 120.65 90)
+      (effects (font (size 1.27 1.27)) hide)
+    )
+    (property "Datasheet" "~" (at 147.32 120.65 0)
+      (effects (font (size 1.27 1.27)) hide)
+    )
+    (property "MPN" "C25744" (at 147.32 120.65 0)
+      (effects (font (size 1.27 1.27)) hide)
+    )
+    (property "JLCPCB Rotation Offset" "" (at 147.32 120.65 0)
+      (effects (font (size 1.27 1.27)) hide)
+    )
+    (pin "1")
+    (pin "2")
+    (instances
+      (project "net-bmp"
+        (path "/0556e588-02fe-48e5-93e8-fa3aab1c90e7"
+          (reference "R9") (unit 1)
+        )
+        (path "/0556e588-02fe-48e5-93e8-fa3aab1c90e7/05fc74b7-f058-42ca-bffa-27bc74c664f2"
+          (reference "R35") (unit 1)
+        )
+      )
