File: hardware/net-bmp/net-bmp.kicad_pcb (KiCad board)
At the start: 4 copper layers, 33.5 x 66.8 mm, 98 parts, among them J1 DBG, J2 Micro SD, J4 USB_C_Receptacle_USB2.0, J5 TGT, J6 BMDU, J7 HR911105A, Q1 DMG1024UV-7, Q2 DMG1024UV-7, SW1 SW_SPST, U1 STM32F407VETx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

Commit message: chore: build with stubs
Parts:
- removed R31: 5.1k, Resistor_SMD:R_0402_1005Metric
- removed R32: 10k, Resistor_SMD:R_0402_1005Metric
- added R35: 10k, Resistor_SMD:R_0402_1005Metric, F.Cu at (151.0, 70.5)
Connections:
- C28 pad 1: +5V -> VBUS
- C29 pad 1: +5V -> VBUS
- J4 pad A4: +5V -> VBUS
- J4 pad A9: +5V -> VBUS
- J4 pad B4: +5V -> VBUS
- J4 pad B9: +5V -> VBUS
- U1 pad 26: /USB_VBUS -> unconnected-(U1-PA3-Pad26)
- U1 pad 68: unconnected-(U1-PA9-Pad68) -> VBUS
- U8 pad 3: +5V -> VBUS
Routing:
- net VBUS: track 0.00 -> 63.3 mm, vias 0 -> 2
- net /USB_VBUS: track 26.7 -> 0.00 mm
- net +5V: track 25.4 -> 0.00 mm
- net /ethernet/LED2: track 28.6 -> 35.1 mm, vias 1 -> 2
- net GND: track 25.6 -> 26.3 mm, vias 54 -> 55
Other:
- board text added: "rev b"
- board text removed: "rev a"
