File: hardware/net-bmp/power.kicad_sch (KiCad schematic)
At the start: 7 parts, among them U3 AMS1117-3.3

Commit message: chore: build with stubs
Connections:
- net +5V renamed VBUS
Changed lines of the file:
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@@
   (title_block
     (title "net-bmp")
-    (date "2023-10-31")
-    (rev "a")
+    (date "2023-11-11")
+    (rev "b")
     (company "elagil")
   )
@@
         (path "/0556e588-02fe-48e5-93e8-fa3aab1c90e7/f869d6ae-fee8-4647-9458-3957901751f8"
           (reference "#FLG06") (unit 1)
+        )
+      )
+    )
+  )
+  (symbol (lib_id "power:VBUS") (at 38.1 35.56 0) (unit 1)
+    (in_bom yes) (on_board yes) (dnp no)
+    (property "Reference" "#PWR067" (at 38.1 39.37 0)
+      (effects (font (size 1.27 1.27)) hide)
+    )
+    (property "Value" "VBUS" (at 38.1 31.75 0)
+      (effects (font (size 1.27 1.27)))
+    )
+    (property "Footprint" "" (at 38.1 35.56 0)
+      (effects (font (size 1.27 1.27)) hide)
+    )
+    (property "Datasheet" "" (at 38.1 35.56 0)
+      (effects (font (size 1.27 1.27)) hide)
+    )
+    (pin "1")
+    (instances
+      (project "net-bmp"
+        (path "/0556e588-02fe-48e5-93e8-fa3aab1c90e7/e157d64e-477b-4983-afb5-0491664aa612"
+          (reference "#PWR067") (unit 1)
+        )
+        (path "/0556e588-02fe-48e5-93e8-fa3aab1c90e7/f869d6ae-fee8-4647-9458-3957901751f8"
+          (reference "#PWR068") (unit 1)
         )
       )
@@
         )
       )
-    )
-  )
-  (symbol (lib_id "power:+5V") (at 38.1 35.56 0) (unit 1)
-    (in_bom yes) (on_board yes) (dnp no) (fields_autoplaced)
-    (property "Reference" "#PWR056" (at 38.1 39.37 0)
-      (effects (font (size 1.27 1.27)) hide)
-    )
-    (property "Value" "+5V" (at 38.1 31.75 0)
-      (effects (font (size 1.27 1.27)))
-    )
-    (property "Footprint" "" (at 38.1 35.56 0)
-      (effects (font (size 1.27 1.27)) hide)
-    )
-    (property "Datasheet" "" (at 38.1 35.56 0)
-      (effects (font (size 1.27 1.27)) hide)
-    )
-    (pin "1")
-    (instances
-      (project "net-bmp"
-        (path "/0556e588-02fe-48e5-93e8-fa3aab1c90e7"
-          (reference "#PWR056") (unit 1)
-        )
-        (path "/0556e588-02fe-48e5-93e8-fa3aab1c90e7/f869d6ae-fee8-4647-9458-3957901751f8"
-          (reference "#PWR071") (unit 1)
-        )
-      )
